Commit message: add joint state simulator

File: examples/nhk2025_sample/urdf/swerve_sample.urdf.xacro (robot description, xacro)
@@ -6,4 +6,5 @@
   <xacro:property name="wheel_radius" value="0.05"/>
   <xacro:property name="wheel_width"  value="0.02"/>
+  <xacro:property name="color_alpha" value="1.0"/>
   <!-- ==================== -->
   <!-- Base link             -->
@@ -20,5 +21,5 @@
       <parent link="base_link"/>
       <child link="${steer_name}_link"/>
-      <origin xyz="${x} ${y} 0" rpy="0 0 0"/>
+      <origin xyz="${x} ${y} ${wheel_radius}" rpy="0 0 0"/>
       <axis xyz="0 0 1"/>
     </joint>
@@ -31,5 +32,5 @@
         <origin rpy="1.5708 0 0"/>
         <material name="black">
-          <color rgba="0.1 0.1 0.1 1.0"/>
+          <color rgba="0.1 0.1 0.1 ${color_alpha}"/>
         </material>
       </visual>
@@ -40,5 +41,5 @@
       <child link="${wheel_name}_link"/>
       <origin xyz="0 0 0" rpy="0 0 0"/>
-      <axis xyz="1 0 0"/>
+      <axis xyz="0 1 0"/>
     </joint>
   </xacro:macro>
@@ -53,8 +54,8 @@
   <!-- Lidar Front          -->
   <!-- ==================== -->
-  <link name="lidar_front_link"/>
+  <link name="lidar_front"/>
   <joint name="base_to_lidar_front" type="fixed">
     <parent link="base_link"/>
-    <child link="lidar_front_link"/>
+    <child link="lidar_front"/>
     <origin xyz="0.4 0 0" rpy="0 0 0"/>
   </joint>
@@ -62,9 +63,9 @@
   <!-- Lidar Rear           -->
   <!-- ==================== -->
-  <link name="lidar_rear_link"/>
+  <link name="lidar_rear"/>
   <joint name="base_to_lidar_rear" type="fixed">
     <parent link="base_link"/>
-    <child link="lidar_rear_link"/>
-    <origin xyz="-0.4 0 0" rpy="0 0 1.5708"/> <!-- rpy = 0 0 pi/2 -->
+    <child link="lidar_rear"/>
+    <origin xyz="-0.4 0 0" rpy="0 0 3.1415926535"/> <!-- rpy = 0 0 pi -->
   </joint>
 </robot>
