Commit message: omni対応

File: examples/nhk2025_sample/urdf/omni_sample.urdf.xacro (robot description, xacro)
@@ -14,12 +14,12 @@
   <!-- Wheel module macro    -->
   <!-- ==================== -->
-  <xacro:macro name="swerve" params="wheel_base_name wheel_name x y">
-    <!-- wheel_base link -->
-    <link name="${wheel_base_name}_link" />
-    <!-- wheel_base joint -->
-    <joint name="${wheel_base_name}" type="continuous">
+  <xacro:macro name="omni" params="wheel_name x y angle">
+    <!-- wheel base link -->
+    <link name="${wheel_name}_base_link"/>
+    <!-- wheel base joint -->
+    <joint name="${wheel_name}_base" type="fixed">
       <parent link="base_link"/>
-      <child link="${wheel_base_name}_link"/>
-      <origin xyz="${x} ${y} ${wheel_radius}" rpy="0 0 0"/>
+      <child link="${wheel_name}_base_link"/>
+      <origin xyz="${x} ${y} ${wheel_radius}" rpy="0 0 ${angle}"/>
       <axis xyz="0 0 1"/>
     </joint>
@@ -38,17 +38,17 @@
     <!-- wheel joint -->
     <joint name="${wheel_name}" type="continuous">
-      <parent link="${wheel_base_name}_link"/>
+      <parent link="${wheel_name}_base_link"/>
       <child link="${wheel_name}_link"/>
-      <origin xyz="0 0 0" rpy="0 0 0"/>
+      <!-- <origin xyz="0 0 0" rpy="0 0 0"/> -->
       <axis xyz="0 1 0"/>
     </joint>
   </xacro:macro>
   <!-- ==================== -->
-  <!-- Wheel instances       -->
+  <!-- Omni instances       -->
   <!-- ==================== -->
-  <xacro:swerve wheel_base_name="swerve_wheel_base_0" wheel_name="swerve_wheel_0" x="0.45"  y="0.45"/>
-  <xacro:swerve wheel_base_name="swerve_wheel_base_1" wheel_name="swerve_wheel_1" x="-0.45" y="0.45"/>
-  <xacro:swerve wheel_base_name="swerve_wheel_base_2" wheel_name="swerve_wheel_2" x="-0.45" y="-0.45"/>
-  <xacro:swerve wheel_base_name="swerve_wheel_base_3" wheel_name="swerve_wheel_3" x="0.45"  y="-0.45"/>
+  <xacro:omni wheel_name="omni_wheel_0" x="0.45"  y="0.45"  angle="-0.7853981635"/>  <!-- angle = -45° -->
+  <xacro:omni wheel_name="omni_wheel_1" x="-0.45" y="0.45"  angle="0.7853981635"/>  <!-- angle = +45° -->
+  <xacro:omni wheel_name="omni_wheel_2" x="-0.45" y="-0.45" angle="2.3561944902"/>  <!-- angle = +135° -->
+  <xacro:omni wheel_name="omni_wheel_3" x="0.45"  y="-0.45" angle="-2.3561944902"/>  <!-- angle = -135° -->
   <!-- ==================== -->
   <!-- Lidar Front          -->
