Commit message: add タイヤが６個あるとスピードが出るんだ

File: examples/nhk2025_sample/urdf/omni_100.urdf.xacro (robot description, xacro)
@@ -47,8 +47,24 @@
   <!-- Omni instances       -->
   <!-- ==================== -->
-  <xacro:omni wheel_name="omni_wheel_0" x="0.45"  y="0.45"  angle="-0.7853981635"/>
-  <xacro:omni wheel_name="omni_wheel_1" x="-0.45" y="0.45"  angle="0.7853981635"/>
-  <xacro:omni wheel_name="omni_wheel_2" x="-0.45" y="-0.45" angle="2.3561944902"/>
-  <xacro:omni wheel_name="omni_wheel_3" x="0.45"  y="-0.45" angle="-2.3561944902"/>
+  <!-- パラメータ -->
+  <xacro:property name="WHEEL_NUM" value="100"/>
+  <xacro:property name="R" value="0.45"/>
+  <xacro:property name="PI" value="3.141592653589793"/>
+ <!-- 再帰マクロ -->
+  <xacro:macro name="omni_loop" params="i">
+    <xacro:if value="${i &lt; WHEEL_NUM}">
+      <xacro:property name="theta"
+        value="${2 * PI * i / WHEEL_NUM}"/>
+      <xacro:omni
+        wheel_name="omni_wheel_${i}"
+        x="${R * cos(theta)}"
+        y="${R * sin(theta)}"
+        angle="${theta + PI / 2}"/>
+      <!-- 次 -->
+      <xacro:omni_loop i="${i + 1}"/>
+    </xacro:if>
+  </xacro:macro>
+  <!-- 開始 -->
+  <xacro:omni_loop i="0"/>
   <!-- ==================== -->
   <!-- Lidar Front          -->

File: examples/nhk2025_sample/urdf/omni_6_high_speed.urdf.xacro (robot description, xacro)
@@ -47,8 +47,16 @@
   <!-- Omni instances       -->
   <!-- ==================== -->
+  <!--
   <xacro:omni wheel_name="omni_wheel_0" x="0.45"  y="0.45"  angle="-0.7853981635"/>
   <xacro:omni wheel_name="omni_wheel_1" x="-0.45" y="0.45"  angle="0.7853981635"/>
   <xacro:omni wheel_name="omni_wheel_2" x="-0.45" y="-0.45" angle="2.3561944902"/>
   <xacro:omni wheel_name="omni_wheel_3" x="0.45"  y="-0.45" angle="-2.3561944902"/>
+  -->
+  <xacro:omni wheel_name="omni_wheel_0" x="0.45"   y="0.0"    angle="1.5707963268"/>   <!--  90° -->
+  <xacro:omni wheel_name="omni_wheel_1" x="0.225"  y="0.3897" angle="2.6179938780"/>   <!-- 150° -->
+  <xacro:omni wheel_name="omni_wheel_2" x="-0.225" y="0.3897" angle="-2.6179938780"/>  <!-- 210° -->
+  <xacro:omni wheel_name="omni_wheel_3" x="-0.45"  y="0.0"    angle="-1.5707963268"/>  <!-- 270° -->
+  <xacro:omni wheel_name="omni_wheel_4" x="-0.225" y="-0.3897" angle="-0.5235987756"/> <!-- 330° -->
+  <xacro:omni wheel_name="omni_wheel_5" x="0.225"  y="-0.3897" angle="0.5235987756"/>  <!--  30° -->
   <!-- ==================== -->
   <!-- Lidar Front          -->
